File: io/ext.kicad_sch (KiCad schematic)
At the start: 53 parts, among them J14 Conn_02x17_Odd_Even, J19 RJ45_Wuerth_7499010121A, J20 AudioJack4_SwitchT1, J21 HDMI_A, Q4 SSM2210, Q5 Q_PNP

Commit message: External I/O
Connections:
- net AUDIO_R_OUT: now reaches J14.15 (Pin_15)
- net AUDIO_L_OUT: now reaches J14.16 (Pin_16)
Changed lines of the file:
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@@
+	(wire
+		(pts
+			(xy 129.54 60.96) (xy 124.46 60.96)
+		)
+		(stroke
+			(width 0)
+			(type default)
+		)
+	)
 	(wire
 		(pts
@@
 		(pts
 			(xy 144.78 43.18) (xy 144.78 48.26)
+		)
+		(stroke
+			(width 0)
+			(type default)
+		)
+	)
+	(wire
+		(pts
+			(xy 142.24 60.96) (xy 147.32 60.96)
 		)
 		(stroke
@@
 	)
 	(global_label "EXT_PWR_ON_N"
-		(shape input)
+		(shape output)
 		(at 147.32 78.74 0)
 		(fields_autoplaced yes)
@@
 	)
 	(hierarchical_label "AV_MODE2"
-		(shape input)
+		(shape output)
 		(at 58.42 195.58 180)
 		(effects
@@
 	)
 	(hierarchical_label "AV_MODE0"
-		(shape input)
+		(shape output)
 		(at 147.32 63.5 0)
 		(effects
@@
 		)
 	)
+	(hierarchical_label "AUDIO_R_OUT"
+		(shape input)
+		(at 124.46 60.96 180)
+		(effects
+			(font
+				(size 1.27 1.27)
+			)
+			(justify right)
+		)
+	)
 	(hierarchical_label "AV_MODE0"
-		(shape input)
+		(shape output)
 		(at 58.42 200.66 180)
 		(effects
@@
 	)
 	(hierarchical_label "AV_MODE1"
-		(shape input)
+		(shape output)
 		(at 147.32 68.58 0)
 		(effects
@@
 	)
 	(hierarchical_label "AV_MODE1"
-		(shape input)
+		(shape output)
 		(at 58.42 198.12 180)
 		(effects
@@
 	)
 	(hierarchical_label "AV_MODE2"
-		(shape input)
+		(shape output)
 		(at 147.32 73.66 0)
 		(effects
@@
 		)
 	)
+	(hierarchical_label "AUDIO_L_OUT"
+		(shape input)
+		(at 147.32 60.96 0)
+		(effects
+			(font
+				(size 1.27 1.27)
+			)
+			(justify left)
+		)
+	)

Commit message: Internal Connectors
Changed lines of the file:
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@@
+		)
+	)
+	(bus
+		(pts
+			(xy 106.68 63.5) (xy 106.68 66.04)
+		)
+		(stroke
+			(width 0)
+			(type default)
 		)
 	)
@@
 	(bus
 		(pts
-			(xy 208.28 201.93) (xy 213.36 201.93)
+			(xy 213.36 199.39) (xy 213.36 201.93)
 		)
 		(stroke
@@
 		)
 	)
+	(bus
+		(pts
+			(xy 187.96 96.52) (xy 187.96 99.06)
+		)
+		(stroke
+			(width 0)
+			(type default)
+		)
+	)
 	(wire
 		(pts
@@
 	(bus
 		(pts
-			(xy 177.8 148.59) (xy 182.88 148.59)
+			(xy 182.88 146.05) (xy 182.88 148.59)
 		)
 		(stroke
@@
 		)
 	)
+	(wire
+		(pts
+			(xy 127 132.08) (xy 127 134.62)
+		)
+		(stroke
+			(width 0)
+			(type default)
+		)
+	)
+	(wire
+		(pts
+			(xy 99.06 104.14) (xy 111.76 104.14)
+		)
+		(stroke
+			(width 0)
+			(type default)
+		)
+	)
+	(wire
+		(pts
+			(xy 198.12 78.74) (xy 203.2 78.74)
+		)
+		(stroke
+			(width 0)
+			(type default)
+		)
+	)
+	(wire
+		(pts
+			(xy 73.66 119.38) (xy 73.66 124.46)
+		)
+		(stroke
+			(width 0)
+			(type default)
+		)
+	)
+	(wire
+		(pts
+			(xy 228.6 78.74) (xy 233.68 78.74)
+		)
+		(stroke
+			(width 0)
+			(type default)
+		)
+	)
 	(bus
 		(pts
-			(xy 182.88 99.06) (xy 187.96 99.06)
-		)
-		(stroke
-			(width 0)
-			(type default)
-		)
-	)
-	(wire
-		(pts
-			(xy 127 132.08) (xy 127 134.62)
-		)
-		(stroke
-			(width 0)
-			(type default)
-		)
-	)
-	(wire
-		(pts
-			(xy 99.06 104.14) (xy 111.76 104.14)
-		)
-		(stroke
-			(width 0)
-			(type default)
-		)
-	)
-	(wire
-		(pts
-			(xy 198.12 78.74) (xy 203.2 78.74)
-		)
-		(stroke
-			(width 0)
-			(type default)
-		)
-	)
-	(wire
-		(pts
-			(xy 73.66 119.38) (xy 73.66 124.46)
-		)
-		(stroke
-			(width 0)
-			(type default)
-		)
-	)
-	(wire
-		(pts
-			(xy 228.6 78.74) (xy 233.68 78.74)
-		)
-		(stroke
-			(width 0)
-			(type default)
-		)
-	)
-	(bus
-		(pts
 			(xy 182.88 153.67) (xy 182.88 151.13)
 		)
@@
 		(pts
 			(xy 233.68 151.13) (xy 233.68 148.59)
-		)
-		(stroke
-			(width 0)
-			(type default)
-		)
-	)
-	(bus
-		(pts
-			(xy 101.6 66.04) (xy 106.68 66.04)
 		)
 		(stroke
@@
 	(hierarchical_label "{HDMI}"
 		(shape bidirectional)
-		(at 101.6 66.04 180)
-		(effects
-			(font
-				(size 1.27 1.27)
-			)
-			(justify right)
+		(at 106.68 63.5 90)
+		(effects
+			(font
+				(size 1.27 1.27)
+			)
+			(justify left)
 		)
 	)
 	(hierarchical_label "{HDMI}"
 		(shape bidirectional)
-		(at 208.28 201.93 180)
-		(effects
-			(font
-				(size 1.27 1.27)
-			)
-			(justify right)
+		(at 213.36 199.39 90)
+		(effects
+			(font
+				(size 1.27 1.27)
+			)
+			(justify left)
 		)
 	)
 	(hierarchical_label "{HDMI}"
 		(shape bidirectional)
-		(at 177.8 148.59 180)
-		(effects
-			(font
-				(size 1.27 1.27)
-			)
-			(justify right)
+		(at 182.88 146.05 90)
+		(effects
+			(font
+				(size 1.27 1.27)
+			)
+			(justify left)
 		)
 	)
@@
 		)
 	)
-	(hierarchical_label "EXPPORT_PORT4{USB}"
+	(hierarchical_label "EXPPORT_PORT3{USB}"
 		(shape bidirectional)
 		(at 218.44 44.45 180)
@@
 	(hierarchical_label "{ETHERNET}"
 		(shape bidirectional)
-		(at 182.88 99.06 180)
-		(effects
-			(font
-				(size 1.27 1.27)
-			)
-			(justify right)
+		(at 187.96 96.52 90)
+		(effects
+			(font
+				(size 1.27 1.27)
+			)
+			(justify left)
 		)
 	)
@@
 		)
 	)
-	(hierarchical_label "EXPPORT_PORT3{USB}"
+	(hierarchical_label "EXPPORT_PORT1{USB}"
 		(shape bidirectional)
-		(at 218.44 41.91 180)
+		(at 218.44 29.21 180)
 		(effects
 			(font
@@
 		)
 	)
-	(hierarchical_label "EXPPORT_PORT1{USB}"
+	(hierarchical_label "EXPPORT_PORT2{USB}"
 		(shape bidirectional)
-		(at 218.44 26.67 180)
+		(at 218.44 41.91 180)
 		(effects
 			(font
@@
 		)
 	)
-	(hierarchical_label "EXPPORT_PORT2{USB}"
+	(hierarchical_label "EXPPORT_PORT0{USB}"
 		(shape bidirectional)
-		(at 218.44 29.21 180)
-		(effects
-			(font
+		(at 218.44 26.67 180)
+		(effects
+			(font

Commit message: Audio Output, Analog isolation and TOSLINK
Parts:
- removed J20: AudioJack4_SwitchT1, symbol Connector_Audio:AudioJack4_SwitchT1
- added C389, C390, C419: 0.1u, symbol Device:C
- added C391: 22p, symbol Device:C
- added D35: D_TVS, symbol Device:D_TVS
- added F7: 1.1A, symbol Device:Polyfuse
- added LED1: TOTX1950A, TOTX1950AF, symbol TOTX1950A:TOTX1950A
- added R185: 5.6k, symbol Device:R
- added TP12: TestPoint_Small, symbol Connector:TestPoint_Small
Connections:
- net GND: now also C389.2, C390.2, C391.2, C419.2, D35.2 (A2), LED1.1 (VSS); no longer D1.2 (A2), D2.2 (A2)
- net SPDIF_OUT: now also C391.1, D35.1 (A1), LED1.4 (INPUT)
- net at J21.13 (CEC): now also TP12.1
- net V_AVIP: now reaches J21.18 (+5V)
- net V_AVIP: now also J14.29 (Pin_29), C389.1, C390.1, C419.1, F7.2, LED1.3 (VCC), R185.1
- new net: LED1.2 (R_LED), R185.2
- new net +5V: F7.1
- new net GNDA: D1.2 (A2), D2.2 (A2)
- no-connect marks 0 -> 1
Other:
- note added: "AV Connector"
- note added: "Back USB"
- note added: "Ethernet"
- note added: "HDMI"
- note added: "Power, Filters and Logic"
- note added: "TOSLINK"
- moved on the sheet: C358, C359, C360, C361, C366, C367, C368, C369, C374, C375, C380, C392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

Commit message: Multipurpose and standby power rails, Reannotated schematic
Added V_1P2, V_1P8, V_5P0DUAL, V_EFUSE, V_GPUPCIE, V_3P3STBY and V_1P2STBY
Parts:
- renumbered C359 to C365, C360 to C366, C366 to C367, C367 to C368, C361 to C369, C368 to C370, C389 to C371, C369 to C372, C358 to C373, C390 to C374, C391 to C375, C419 to C376, C357 to C377, C374 to C378, C375 to C379, C392 to C381, D28 to D10, D25 to D11, D31 to D12, D27 to D13, D26 to D14, D32 to D15, D7 to D16, D1 to D3, D30 to D4, D23 to D5, D29 to D6, D24 to D7, D35 to D8, D33 to D9, F7 to F1, FB14 to FB16, J14 to J5, J21 to J6, J19 to J7, Q4 to Q3, Q5 to Q4, R93 to R140, R92 to R141, R102 to R142, R103 to R143, R108 to R144, R117 to R145, R104 to R146, R105 to R147, R109 to R148, R118 to R149, R110 to R150, R119 to R151, R106 to R152, R120 to R153, R107 to R154, R136 to R155, R135 to R156, R138 to R157, R137 to R158, R185 to R159, TP12 to TP39
